File: hardware/CANdiy-FD-Shield_v11.brd (EAGLE design)
At the start: 68.6 x 53.3 mm, 59 parts, among them IC1 MCP2517FDT-H/SL, IC3 MCP2562FDT-E/SN, Q1 16MHz, U1 UNO_ISP, X1 PASSER-07, X2 PASSER-07, X3 PASSER-07

Commit message: updated schematics
Parts:
- Q1: value 16MHz -> 20MHz
Changed lines of the file:
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@@
 <element name="IC3" library="we-chip" package="SO08" value="MCP2562FDT-E/SN" x="20.955" y="28.35275" rot="R270"/>
 <element name="IC1" library="we-chip" package="SO14" value="MCP2517FDT-H/SL" x="20.79625" y="38.1" rot="R180"/>
-<element name="Q1" library="we-rcl" package="CRYSTAL_32X13" value="16MHz" x="22.70125" y="43.815" rot="R270"/>
+<element name="Q1" library="we-rcl" package="CRYSTAL_32X13" value="20MHz" x="22.70125" y="43.815" rot="R270"/>
 <element name="D1" library="we-rcl" package="SOD323" value="" x="8.89" y="5.461" rot="R270"/>
 </elements>
